Commit message: ok xbot dummy mode

File: frankapanda_urdf/urdf/common/franka_robot.xacro (robot description, xacro)
@@ -14,5 +14,13 @@
     <xacro:include filename="$(find frankapanda_urdf)/urdf/common/franka_arm.xacro" />
     <xacro:franka_arm arm_id="${arm_id}" safety_distance="0.03" gazebo="$(arg gazebo)" joint_limits="${joint_limits}"/>
-    <xacro:if value="$(arg hand)">
+    <xacro:if value="${END_EFFECTOR == 'none'}">
+      <link name="tcp" />
+      <joint name="j_tcp" type="fixed">
+          <parent link="${arm_id}_link8" />
+          <child link="tcp" />
+          <origin xyz="0 0 0" rpy="0 0 0"/>
+      </joint>
+    </xacro:if>
+    <xacro:if value="${END_EFFECTOR == 'panda_hand'}">
       <xacro:include filename="$(find frankapanda_urdf)/urdf/common/franka_hand.xacro"/>
       <xacro:franka_hand
@@ -24,5 +32,11 @@
           safety_distance="0.03"
           gazebo="$(arg gazebo)"
-       />
+      />
+      <link name="tcp" />
+      <joint name="j_tcp" type="fixed">
+          <parent link="${arm_id}_hand_tcp" />
+          <child link="tcp" />
+          <origin xyz="0 0 0" rpy="0 0 0"/>
+      </joint>
     </xacro:if>
     <!-- Define additional Gazebo tags -->

File: frankapanda_urdf/urdf/panda.urdf.xacro (robot description, xacro)
@@ -2,5 +2,5 @@
 <robot xmlns:xacro="http://www.ros.org/wiki/xacro" name="panda">
   <xacro:include filename="$(find frankapanda_urdf)/urdf/common/franka_robot.xacro"/>
-  <xacro:arg name="arm_id" default="panda" />
+  <xacro:include filename="$(find frankapanda_urdf)/config/frankapanda.urdf.xacro"/>
   <xacro:franka_robot arm_id="$(arg arm_id)"
                       joint_limits="${xacro.load_yaml('$(find franka_description)/robots/panda/joint_limits.yaml')}">
