Commit message: ros2 port

File: frankapanda_urdf/urdf/common/utils.xacro (robot description, xacro)
@@ -38,10 +38,10 @@
       <visual>
         <geometry>
-          <mesh filename="package://${description_pkg}/meshes/visual/${name}.dae" />
+          <mesh filename="file://$(find frankapanda_urdf)/meshes/visual/${name}.dae" />
         </geometry>
       </visual>
       <collision>
         <geometry>
-          <mesh filename="package://${description_pkg}/meshes/collision/${name}.stl" />
+          <mesh filename="file://$(find frankapanda_urdf)/meshes/collision/${name}.stl" />
         </geometry>
       </collision>

File: frankapanda_urdf/urdf/common/xbot.gazebo.xacro (robot description, xacro)
@@ -1,33 +1,47 @@
 <?xml version="1.0"?>
-<robot xmlns:xacro="http://ros.org/wiki/xacro">
+<robot xmlns:xacro="http://ros.org/wiki/xacro" name="frankapanda">
 <gazebo>
-    <plugin name="xbot2_joint_driver" filename="libxbot2_gz_joint_server.so">
-        <pid>
+    <plugin filename="xbot2_gz_joint_server"
+            name="gz::sim::systems::GzJointServer">
         <!-- gains from https://github.com/frankaemika/franka_ros/blob/develop/franka_gazebo/config/franka_hw_sim.yaml -->
-            <gain name="very_small_mot"  p="50"  d="5"/>
-            <gain name="small_mot"  p="600"  d="6"/>
-            <gain name="medium_mot" p="7000" d="50"/>
-            <gain name="big_mot"    p="8000" d="50"/>
+        <profile name="very_small_mot"  p="50"  d="5"/>
+        <profile name="small_mot"  p="600"  d="6"/>
+        <profile name="medium_mot" p="7000" d="50"/>
+        <profile name="big_mot"    p="8000" d="50"/>
+        <xacro:if value="${END_EFFECTOR == 'dagana'}">
+            <profile name="dagana_mot"  p="10" d="0.5"/>
+        </xacro:if>
+        <xacro:if value="${END_EFFECTOR == 'panda_hand'}">
+            <profile name="fingers_mot"  p="100" d="1"/>
+        </xacro:if>
+        <pid name="${arm_id}_joint1" profile="medium_mot"/>
+        <pid name="${arm_id}_joint2" profile="medium_mot"/>
+        <pid name="${arm_id}_joint3" profile="medium_mot"/>
+        <pid name="${arm_id}_joint4" profile="medium_mot"/>
+        <pid name="${arm_id}_joint5" profile="medium_mot"/>
+        <pid name="${arm_id}_joint6" profile="medium_mot"/>
+        <pid name="${arm_id}_joint7" profile="small_mot"/>
+        <xacro:if value="${END_EFFECTOR == 'dagana'}">
+            <pid name="dagana_1_claw_joint" profile="dagana_mot"/>
+        </xacro:if>
+        <xacro:if value="${END_EFFECTOR == 'panda_hand'}">
+            <pid name="${arm_id}_finger_joint1" profile="fingers_mot"/>
+            <pid name="${arm_id}_finger_joint2" profile="fingers_mot"/>
+        </xacro:if>
+        <initial_configuration>
+            <joint name="joint_1" value="0"/>
+            <joint name="joint_2" value="0"/>
+            <joint name="joint_3" value="0"/>
+            <joint name="joint_4" value="0"/>
+            <joint name="joint_5" value="0"/>
+            <joint name="joint_6" value="0"/>
             <xacro:if value="${END_EFFECTOR == 'dagana'}">
-                <gain name="dagana_mot"  p="10" d="0.5"/>
+                <joint name="dagana_1_claw_joint" value="0"/>
             </xacro:if>
             <xacro:if value="${END_EFFECTOR == 'panda_hand'}">
-                <gain name="fingers_mot"  p="100" d="1"/>
+                <pid name="${arm_id}_finger_joint1" value="0"/>
+                <pid name="${arm_id}_finger_joint2" value="0"/>
             </xacro:if>
-            <pid name="${arm_id}_joint1" profile="medium_mot"/>
-            <pid name="${arm_id}_joint2" profile="medium_mot"/>
-            <pid name="${arm_id}_joint3" profile="medium_mot"/>
-            <pid name="${arm_id}_joint4" profile="medium_mot"/>
-            <pid name="${arm_id}_joint5" profile="medium_mot"/>
-            <pid name="${arm_id}_joint6" profile="medium_mot"/>
-            <pid name="${arm_id}_joint7" profile="small_mot"/>
-            <xacro:if value="${END_EFFECTOR == 'dagana'}">
-                <pid name="dagana_1_claw_joint" profile="dagana_mot"/>
-            </xacro:if>
-            <xacro:if value="${END_EFFECTOR == 'panda_hand'}">
-                <pid name="${arm_id}_finger_joint1" profile="fingers_mot"/>
-                <pid name="${arm_id}_finger_joint2" profile="fingers_mot"/>
-            </xacro:if>
-        </pid>
+        </initial_configuration>
     </plugin>
 </gazebo>
