Commit message: working in gazebo sim with xbot && dagana option

File: frankapanda_srdf/srdf/panda.srdf.xacro (robot description, xacro)
@@ -6,4 +6,9 @@
         <chain base_link="${arm_id}_link0" tip_link="tcp"/>
     </group>
+    <xacro:if value="${END_EFFECTOR == 'dagana'}">
+        <group name="dagana">
+            <chain base_link="${arm_id}_link8" tip_link="dagana_1_bottom_link"/>
+        </group>
+    </xacro:if>
     <xacro:if value="${END_EFFECTOR == 'panda_hand'}">
         <group name="${arm_id}_finger1">
@@ -17,4 +22,7 @@
 	<group name="chains">
 		<group name="arm"/>
+        <xacro:if value="${END_EFFECTOR == 'dagana'}">
+            <group name="dagana"></group>
+        </xacro:if>
         <xacro:if value="${END_EFFECTOR == 'panda_hand'}">
             <group name="${arm_id}_finger1"/>

File: frankapanda_urdf/config/frankapanda.urdf.xacro (robot description, xacro)
@@ -5,7 +5,7 @@
 <xacro:arg name="arm_id" default="panda" />
 <xacro:property name="arm_id" value="$(arg arm_id)" />
-<xacro:arg name="gazebo" default="true" />
+<xacro:arg name="gazebo" default="false" />
 <xacro:property name="gazebo" value="$(arg gazebo)" />
-<xacro:arg name="end_effector" default="panda_hand"/> <!-- none, panda_hand, dagana_fixed, dagana -->
+<xacro:arg name="end_effector" default="panda_hand"/> <!-- none, panda_hand, dagana -->
 <xacro:property name="END_EFFECTOR" value="$(arg end_effector)" />
 </robot>

File: frankapanda_urdf/urdf/common/franka_arm.xacro (robot description, xacro)
@@ -1,8 +1,8 @@
 <?xml version='1.0' encoding='utf-8'?>
 <robot xmlns:xacro="http://www.ros.org/wiki/xacro" name="panda">
-  <xacro:include filename="$(find franka_description)/robots/common/utils.xacro" />
+  <xacro:include filename="$(find frankapanda_urdf)/urdf/common/utils.xacro" />
   <!-- safety_distance: Minimum safety distance in [m] by which the collision volumes are expanded and which is enforced during robot motions -->
   <!-- arm_id: Namespace of the robot arm. Serves to differentiate between arms in case of multiple instances. -->
-  <!-- joint_limits: description of the joint limits that comes from a YAML file. Example definition: ${xacro.load_yaml('$(find franka_description)/robots/fr3/joint_limits.yaml')} -->
+  <!-- joint_limits: description of the joint limits that comes from a YAML file. Example definition: ${xacro.load_yaml('$(find frankapanda_urdf)/urdf/joint_limits.yaml')} -->
   <xacro:macro name="franka_arm" params="arm_id:='panda' description_pkg:='frankapanda_urdf' connected_to:='' xyz:='0 0 0' rpy:='0 0 0' gazebo:=false safety_distance:=0 joint_limits" >
     <xacro:unless value="${not connected_to}">

File: frankapanda_urdf/urdf/common/franka_robot.xacro (robot description, xacro)
@@ -2,10 +2,7 @@
 <robot xmlns:xacro="http://www.ros.org/wiki/xacro">
   <xacro:macro name="franka_robot" params="arm_id joint_limits">
-    <!-- Name of this panda -->
-    <!-- Should a franka_gripper be mounted at the flange?" -->
-    <xacro:arg name="hand" default="false" />
-    <!-- Positional offset between $(arm_id)_hand -> $(arm_id)_hand_tcp [m]. Only used when hand:=true -->
+    <!-- Positional offset between $(arm_id)_hand -> $(arm_id)_hand_tcp [m]. Only used when END_EFFECTOR:=panda_hand -->
     <xacro:arg name="tcp_xyz" default="0 0 0.1034" />
-    <!-- Rotational offset between $(arm_id)_hand -> $(arm_id)_hand_tcp [rad]. Only used when hand:=true -->
+    <!-- Rotational offset between $(arm_id)_hand -> $(arm_id)_hand_tcp [rad]. Only used when END_EFFECTOR:=panda_hand -->
     <xacro:arg name="tcp_rpy" default="0 0 0" />
     <!-- Is the robot being simulated in gazebo?" -->
@@ -22,4 +19,17 @@
       </joint>
     </xacro:if>
+    <xacro:if value="${END_EFFECTOR == 'dagana'}">
+        <xacro:include filename="$(find dagana_urdf)/urdf/dagana_macro.urdf.xacro" />
+        <xacro:dagana_gripper name="dagana_1" parent_link="${arm_id}_link8" joint_type="revolute">
+            <origin xyz="0 0 0" rpy="0 0 0"/>
+        </xacro:dagana_gripper>
+        <!--     to have the same final link as when "none" option is used     -->
+        <link name="tcp" />
+        <joint name="j_tcp" type="fixed">
+            <parent link="dagana_1_tcp" />
+            <child link="tcp" />
+            <origin xyz="0 0 0" rpy="0 0 0"/>
+        </joint>
+    </xacro:if>
     <xacro:if value="${END_EFFECTOR == 'panda_hand'}">
       <xacro:include filename="$(find frankapanda_urdf)/urdf/common/franka_hand.xacro"/>
@@ -33,4 +43,11 @@
           gazebo="$(arg gazebo)"
       />
+      <xacro:if value="$(arg gazebo)">
+        <xacro:gazebo-joint joint="${arm_id}_finger_joint1" />
+        <xacro:gazebo-joint joint="${arm_id}_finger_joint2"  />
+        <!-- Friction specific material for Rubber/Rubber contact -->
+        <xacro:gazebo-friction link="${arm_id}_leftfinger" mu="1.13" />
+        <xacro:gazebo-friction link="${arm_id}_rightfinger" mu="1.13" />
+      </xacro:if>
       <link name="tcp" />
       <joint name="j_tcp" type="fixed">
@@ -42,13 +59,4 @@
     <!-- Define additional Gazebo tags -->
     <xacro:if value="$(arg gazebo)">
-      <xacro:arg name="xyz" default="0 0 0" />
-      <xacro:arg name="rpy" default="0 0 0" />
-      <!-- Gazebo requires a joint to a link called "world" for statically mounted robots -->
-      <link name="world" />
-      <joint name="world_joint" type="fixed">
-        <origin xyz="$(arg xyz)" rpy="$(arg rpy)" />
-        <parent link="world" />
-        <child  link="$(arg arm_id)_link0" />
-      </joint>
       <xacro:gazebo-joint joint="${arm_id}_joint1"  />
       <xacro:gazebo-joint joint="${arm_id}_joint2"  />
@@ -58,11 +66,4 @@
       <xacro:gazebo-joint joint="${arm_id}_joint6"  />
       <xacro:gazebo-joint joint="${arm_id}_joint7"  />
-      <xacro:if value="$(arg hand)">
-        <xacro:gazebo-joint joint="${arm_id}_finger_joint1" />
-        <xacro:gazebo-joint joint="${arm_id}_finger_joint2"  />
-        <!-- Friction specific material for Rubber/Rubber contact -->
-        <xacro:gazebo-friction link="${arm_id}_leftfinger" mu="1.13" />
-        <xacro:gazebo-friction link="${arm_id}_rightfinger" mu="1.13" />
-      </xacro:if>
       <xacro:include filename="$(find frankapanda_urdf)/urdf/common/xbot.gazebo.xacro" />
     </xacro:if>

File: frankapanda_urdf/urdf/common/xbot.gazebo.xacro (robot description, xacro)
@@ -1,5 +1,4 @@
 <?xml version="1.0"?>
 <robot xmlns:xacro="http://ros.org/wiki/xacro">
-<xacro:macro name="xbot2_joint_driver_macro" params="arm_id">
 <gazebo>
     <plugin name="xbot2_joint_driver" filename="libxbot2_gz_joint_server.so">
@@ -10,6 +9,10 @@
             <gain name="medium_mot" p="250" d="10"/>
             <gain name="big_mot"    p="600" d="30"/>
-            <gain name="dagana_mot"  p="10" d="0.5"/>
-            <gain name="fingers_mot"  p="100" d="1"/>
+            <xacro:if value="${END_EFFECTOR == 'dagana'}">
+                <gain name="dagana_mot"  p="10" d="0.5"/>
+            </xacro:if>
+            <xacro:if value="${END_EFFECTOR == 'panda_hand'}">
+                <gain name="fingers_mot"  p="100" d="1"/>
+            </xacro:if>
             <pid name="${arm_id}_joint1" profile="small_mot"/>
             <pid name="${arm_id}_joint2" profile="small_mot"/>
@@ -19,10 +22,13 @@
             <pid name="${arm_id}_joint6" profile="small_mot"/>
             <pid name="${arm_id}_joint7" profile="small_mot"/>
-            <pid name="dagana_1_claw_joint" profile="dagana_mot"/>
-            <pid name="${arm_id}_finger_joint1" profile="fingers_mot"/>
-            <pid name="${arm_id}_finger_joint2" profile="fingers_mot"/>
+            <xacro:if value="${END_EFFECTOR == 'dagana'}">
+                <pid name="dagana_1_claw_joint" profile="dagana_mot"/>
+            </xacro:if>
+            <xacro:if value="${END_EFFECTOR == 'panda_hand'}">
+                <pid name="${arm_id}_finger_joint1" profile="fingers_mot"/>
+                <pid name="${arm_id}_finger_joint2" profile="fingers_mot"/>
+            </xacro:if>
         </pid>
     </plugin>
 </gazebo>
-</xacro:macro>
 </robot>

File: frankapanda_urdf/urdf/panda.urdf.xacro (robot description, xacro)
@@ -3,6 +3,27 @@
   <xacro:include filename="$(find frankapanda_urdf)/urdf/common/franka_robot.xacro"/>
   <xacro:include filename="$(find frankapanda_urdf)/config/frankapanda.urdf.xacro"/>
+  <xacro:arg name="x" default="0"/>
+  <xacro:arg name="y" default="0"/>
+  <xacro:arg name="z" default="0"/>
+  <xacro:arg name="roll" default="0"/>
+  <xacro:arg name="pitch" default="0"/>
+  <xacro:arg name="yaw" default="0"/>
+  <xacro:if value="$(arg gazebo)">
+    <xacro:arg name="parent" default="world"/>
+    <link name="$(arg parent)" />
+  </xacro:if>
+  <xacro:unless value="$(arg gazebo)">
+    <xacro:arg name="parent" default=""/>
+  </xacro:unless>
+  <xacro:property name="parent" value="$(arg parent)"/>
+  <xacro:unless value="${parent == ''}">
+    <joint name="${parent}_joint" type="fixed">
+        <parent link="${parent}" />
+        <child link="$(arg arm_id)_link0" />
+        <origin xyz="$(arg x) $(arg y) $(arg z)" rpy="$(arg roll) $(arg pitch) $(arg yaw)"/>
+    </joint>
+  </xacro:unless>
   <xacro:franka_robot arm_id="$(arg arm_id)"
-                      joint_limits="${xacro.load_yaml('$(find franka_description)/robots/panda/joint_limits.yaml')}">
+                      joint_limits="${xacro.load_yaml('$(find frankapanda_urdf)/urdf/joint_limits.yaml')}">
   </xacro:franka_robot>
 </robot>

Commit message: nicla and dagana in srdf

File: frankapanda_srdf/srdf/panda.srdf.xacro (robot description, xacro)
@@ -39,4 +39,30 @@
 		<joint name="${arm_id}_joint6" value="1.3"/>
 		<joint name="${arm_id}_joint7" value="0"/>
+        <xacro:if value="${END_EFFECTOR == 'panda_hand'}">
+		    <joint name="${arm_id}_finger_joint1" value="0"/>
+		    <joint name="${arm_id}_finger_joint2" value="0"/>
+        </xacro:if>
+        <xacro:if value="${END_EFFECTOR == 'dagana'}">
+            <joint name="dagana_1_claw_joint" value="0"/>
+        </xacro:if>
 	</group_state>
+    <!--DISABLE COLLISIONS: By default it is assumed that any link of the robot could potentially come into collision with any other link in the robot. This tag disables collision checking between a specified pair of links. -->
+    <disable_collisions link1="${arm_id}_link0" link2="${arm_id}_link1" reason="Adjacent"/>
+    <disable_collisions link1="${arm_id}_link1" link2="${arm_id}_link2" reason="Adjacent"/>
+    <disable_collisions link1="${arm_id}_link2" link2="${arm_id}_link3" reason="Adjacent"/>
+    <disable_collisions link1="${arm_id}_link3" link2="${arm_id}_link4" reason="Adjacent"/>
+    <disable_collisions link1="${arm_id}_link4" link2="${arm_id}_link5" reason="Adjacent"/>
+    <disable_collisions link1="${arm_id}_link5" link2="${arm_id}_link6" reason="Adjacent"/>
+    <disable_collisions link1="${arm_id}_link6" link2="${arm_id}_link7" reason="Adjacent"/>
+    <xacro:if value="${END_EFFECTOR == 'dagana'}">
+        <disable_collisions link1="${arm_id}_link6" link2="dagana_1_bottom_link" reason="Never"/>
+        <disable_collisions link1="${arm_id}_link6" link2="dagana_1_top_link" reason="Never"/>
+        <disable_collisions link1="${arm_id}_link7" link2="dagana_1_bottom_link" reason="Adjacent"/>
+        <disable_collisions link1="${arm_id}_link7" link2="dagana_1_top_link" reason="Adjacent"/>
+        <disable_collisions link1="dagana_1_bottom_link" link2="dagana_1_top_link" reason="Adjacent"/>
+        <xacro:if value="${NICLA}">
+            <disable_collisions link1="dagana_1_bottom_link" link2="nicla_base" reason="Adjacent"/>
+            <disable_collisions link1="dagana_1_top_link" link2="nicla_base" reason="Adjacent"/>
+        </xacro:if>
+    </xacro:if>
 </robot>

File: frankapanda_urdf/config/frankapanda.urdf.xacro (robot description, xacro)
@@ -11,3 +11,5 @@
 <xacro:arg name="end_effector" default="panda_hand"/> <!-- none, panda_hand, dagana -->
 <xacro:property name="END_EFFECTOR" value="$(arg end_effector)" />
+<xacro:arg name="nicla" default="false"/> <!-- the nicla inside the dagana-->
+<xacro:property name="NICLA" value="$(arg nicla)" />
 </robot>

Commit message: unbug

File: frankapanda_srdf/srdf/panda.srdf.xacro (robot description, xacro)
@@ -55,4 +55,7 @@
     <disable_collisions link1="${arm_id}_link5" link2="${arm_id}_link6" reason="Adjacent"/>
     <disable_collisions link1="${arm_id}_link6" link2="${arm_id}_link7" reason="Adjacent"/>
+    <xacro:if value="${USE_ROUND_BASE}">
+        <disable_collisions link1="${arm_id}_round_base_link" link2="${arm_id}_link0" reason="Adjacent"/>
+    </xacro:if>
     <xacro:if value="${END_EFFECTOR == 'dagana'}">
         <disable_collisions link1="${arm_id}_link6" link2="dagana_1_bottom_link" reason="Never"/>

File: frankapanda_urdf/urdf/panda.urdf.xacro (robot description, xacro)
@@ -48,6 +48,6 @@
       </collision>
       <xacro:if value="$(arg gazebo)">
-        <xacro:cylinder_inertial mass="1" length="0.10" radius="0.1">
-            <origin xyz="0 0 0.05" rpy="0 0 0" />
+        <xacro:cylinder_inertial mass="1" length="0.02" radius="0.15">
+            <origin xyz="0 0 0.01" rpy="0 0 0" />
         </xacro:cylinder_inertial>
       </xacro:if>

Commit message: adapter mounting for dagana

File: frankapanda_srdf/srdf/panda.srdf.xacro (robot description, xacro)
@@ -64,7 +64,11 @@
         <disable_collisions link1="${arm_id}_link7" link2="dagana_1_top_link" reason="Adjacent"/>
         <disable_collisions link1="dagana_1_bottom_link" link2="dagana_1_top_link" reason="Adjacent"/>
+        <disable_collisions link1="dagana_mount" link2="dagana_1_top_link" reason="Adjacent"/>
+        <disable_collisions link1="dagana_mount" link2="dagana_1_bottom_link" reason="Adjacent"/>
+        <disable_collisions link1="${arm_id}_link7" link2="dagana_mount" reason="Adjacent"/>
         <xacro:if value="${NICLA}">
             <disable_collisions link1="dagana_1_bottom_link" link2="nicla_base" reason="Adjacent"/>
             <disable_collisions link1="dagana_1_top_link" link2="nicla_base" reason="Adjacent"/>
+            <disable_collisions link1="dagana_mount" link2="nicla_base" reason="Adjacent"/>
         </xacro:if>
     </xacro:if>

File: frankapanda_urdf/config/frankapanda.urdf.xacro (robot description, xacro)
@@ -13,3 +13,6 @@
 <xacro:arg name="nicla" default="false"/> <!-- the nicla inside the dagana-->
 <xacro:property name="NICLA" value="$(arg nicla)" />
+<material name="mount_dagana_dark_grey">
+	<color rgba="0.2 0.2 0.2 1"/>
+</material>
 </robot>

File: frankapanda_urdf/urdf/common/franka_robot.xacro (robot description, xacro)
@@ -29,5 +29,27 @@
     <xacro:if value="${END_EFFECTOR == 'dagana'}">
         <xacro:include filename="$(find dagana_urdf)/urdf/dagana_macro.urdf.xacro" />
-        <xacro:dagana_gripper name="dagana_1" parent_link="${arm_id}_link8" joint_type="revolute">
+        <link name="dagana_mount">
+          <visual>
+            <geometry>
+              <mesh filename="package://frankapanda_urdf/meshes/visual/ce0327_iso-adapter.stl" scale="0.001 0.001 0.001"/>
+            </geometry>
+            <material name="mount_dagana_dark_grey"/>
+          </visual>
+          <collision>
+            <geometry>
+              <mesh filename="package://frankapanda_urdf/meshes/visual/ce0327_iso-adapter.stl" scale="0.001 0.001 0.001"/>
+            </geometry>
+          </collision>
+          <!-- TODO put real inertia -->
+          <xacro:cylinder_inertial mass="0.200" length="0.027" radius="0.10">
+            <origin xyz="0 0 0" rpy="0 0 0" />
+          </xacro:cylinder_inertial>
+        </link>
+        <joint name="${arm_id}_link8_to_dagana" type="fixed">
+            <parent link="${arm_id}_link8" />
+            <child link="dagana_mount" />
+            <origin xyz="0 0 0.00135" rpy="0 0 0"/>
+        </joint>
+        <xacro:dagana_gripper name="dagana_1" parent_link="dagana_mount" joint_type="revolute">
             <origin xyz="0 0 0" rpy="0 0 0"/>
         </xacro:dagana_gripper>
