Commit message: dagana use and round base we use in lab

File: frankapanda_urdf/config/frankapanda.urdf.xacro (robot description, xacro)
@@ -7,4 +7,6 @@
 <xacro:arg name="gazebo" default="false" />
 <xacro:property name="gazebo" value="$(arg gazebo)" />
+<xacro:arg name="use_round_base" default="true"/>
+<xacro:property name="USE_ROUND_BASE" value="$(arg use_round_base)" />
 <xacro:arg name="end_effector" default="panda_hand"/> <!-- none, panda_hand, dagana -->
 <xacro:property name="END_EFFECTOR" value="$(arg end_effector)" />

File: frankapanda_urdf/urdf/common/franka_robot.xacro (robot description, xacro)
@@ -1,5 +1,5 @@
 <?xml version='1.0' encoding='utf-8'?>
 <robot xmlns:xacro="http://www.ros.org/wiki/xacro">
-  <xacro:macro name="franka_robot" params="arm_id joint_limits">
+  <xacro:macro name="franka_robot" params="arm_id joint_limits parent='' xyz:='0 0 0' rpy:='0 0 0'">
     <!-- Positional offset between $(arm_id)_hand -> $(arm_id)_hand_tcp [m]. Only used when END_EFFECTOR:=panda_hand -->
     <xacro:arg name="tcp_xyz" default="0 0 0.1034" />
@@ -10,5 +10,13 @@
     <xacro:include filename="$(find frankapanda_urdf)/urdf/common/utils.xacro" />
     <xacro:include filename="$(find frankapanda_urdf)/urdf/common/franka_arm.xacro" />
-    <xacro:franka_arm arm_id="${arm_id}" safety_distance="0.03" gazebo="$(arg gazebo)" joint_limits="${joint_limits}"/>
+    <xacro:franka_arm
+      arm_id="${arm_id}"
+      safety_distance="0.03"
+      gazebo="$(arg gazebo)"
+      joint_limits="${joint_limits}"
+      connected_to="${parent}"
+      xyz="${xyz}"
+      rpy="${rpy}"
+    />
     <xacro:if value="${END_EFFECTOR == 'none'}">
       <link name="tcp" />

File: frankapanda_urdf/urdf/common/utils.xacro (robot description, xacro)
@@ -148,4 +148,13 @@
     </inertial>
   </xacro:macro>
+  <xacro:macro name="cylinder_inertial" params="radius length mass *origin">
+      <inertial>
+      <mass value="${mass}" />
+      <xacro:insert_block name="origin" />
+      <inertia ixx="${0.0833333 * mass * (3 * radius * radius + length * length)}" ixy="0.0" ixz="0.0"
+          iyy="${0.0833333 * mass * (3 * radius * radius + length * length)}" iyz="0.0"
+          izz="${0.5 * mass * radius * radius}" />
+      </inertial>
+  </xacro:macro>
   <!-- ========================================================================= -->
   <!-- Adds the <limit ... /> & <safety_controller/> tags given a config file    -->

File: frankapanda_urdf/urdf/panda.urdf.xacro (robot description, xacro)
@@ -2,4 +2,5 @@
 <robot xmlns:xacro="http://www.ros.org/wiki/xacro" name="panda">
   <xacro:include filename="$(find frankapanda_urdf)/urdf/common/franka_robot.xacro"/>
+  <xacro:include filename="$(find frankapanda_urdf)/urdf/common/utils.xacro"/>
   <xacro:include filename="$(find frankapanda_urdf)/config/frankapanda.urdf.xacro"/>
   <xacro:arg name="x" default="0"/>
@@ -20,10 +21,46 @@
     <joint name="${parent}_joint" type="fixed">
         <parent link="${parent}" />
-        <child link="$(arg arm_id)_link0" />
+        <xacro:if value="${USE_ROUND_BASE}">
+          <child link="$(arg arm_id)_round_base_link" />
+        </xacro:if>
+        <xacro:unless value="${USE_ROUND_BASE}">
+          <child link="$(arg arm_id)_link0" />
+        </xacro:unless>
         <origin xyz="$(arg x) $(arg y) $(arg z)" rpy="$(arg roll) $(arg pitch) $(arg yaw)"/>
     </joint>
   </xacro:unless>
-  <xacro:franka_robot arm_id="$(arg arm_id)"
-                      joint_limits="${xacro.load_yaml('$(find frankapanda_urdf)/urdf/joint_limits.yaml')}">
-  </xacro:franka_robot>
+  <xacro:if value="${USE_ROUND_BASE}">
+    <link name="$(arg arm_id)_round_base_link">
+      <visual>
+        <origin xyz="0 0 0.01" rpy="0 0 0" />
+        <geometry>
+          <cylinder radius="0.15" length="0.02"/>
+        </geometry>
+        <material name="panda_round_base_link_material">
+          <color rgba="0.4431 0.47 0.494 1"/>
+        </material>
+      </visual>
+      <collision>
+        <origin xyz="0 0 0.01" rpy="0 0 0" />
+        <geometry>
+          <cylinder radius="0.15" length="0.02"/>
+        </geometry>
+      </collision>
+      <xacro:if value="$(arg gazebo)">
+        <xacro:cylinder_inertial mass="1" length="0.10" radius="0.1">
+            <origin xyz="0 0 0.05" rpy="0 0 0" />
+        </xacro:cylinder_inertial>
+      </xacro:if>
+    </link>
+    <xacro:franka_robot arm_id="$(arg arm_id)"
+                        joint_limits="${xacro.load_yaml('$(find frankapanda_urdf)/urdf/joint_limits.yaml')}"
+                        parent="$(arg arm_id)_round_base_link"
+                        xyz="0.05 0.004 0.02">
+    </xacro:franka_robot>
+  </xacro:if>
+  <xacro:unless value="${USE_ROUND_BASE}">
+    <xacro:franka_robot arm_id="$(arg arm_id)"
+                        joint_limits="${xacro.load_yaml('$(find frankapanda_urdf)/urdf/joint_limits.yaml')}">
+    </xacro:franka_robot>
+  </xacro:unless>
 </robot>

Commit message: safety distance as argument

File: frankapanda_urdf/config/frankapanda.urdf.xacro (robot description, xacro)
@@ -13,4 +13,6 @@
 <xacro:arg name="nicla" default="false"/> <!-- the nicla inside the dagana-->
 <xacro:property name="NICLA" value="$(arg nicla)" />
+<xacro:arg name="safety_distance" default="0.03"/> <!-- for collision meshes, used only when gazebo:=false (I do not know why)-->
+<xacro:property name="SAFETY_DISTANCE" value="$(arg safety_distance)" />
 <material name="mount_dagana_dark_grey">
 	<color rgba="0.2 0.2 0.2 1"/>

File: frankapanda_urdf/urdf/common/franka_robot.xacro (robot description, xacro)
@@ -12,5 +12,5 @@
     <xacro:franka_arm
       arm_id="${arm_id}"
-      safety_distance="0.03"
+      safety_distance="${SAFETY_DISTANCE}"
       gazebo="$(arg gazebo)"
       joint_limits="${joint_limits}"
